Commit message: Adding IsaacSim

File: jetauto/jetauto_description/urdf/jetauto_car.urdf.xacro (robot description, xacro)
@@ -111,5 +111,5 @@
   <joint
     name="wheel_right_front_joint"
-    type="fixed">
+    type="continuous">
     <origin
       xyz="0.097397 -0.086125 0.04508"
@@ -119,4 +119,5 @@
     <child
       link="wheel_right_front_link" />
+    <axis xyz="0 0 1" />
   </joint>
   <link
@@ -144,5 +145,5 @@
   <joint
     name="wheel_left_front_joint"
-    type="fixed">
+    type="continuous">
     <origin
       xyz="0.097397 0.086125 0.04508"
@@ -152,4 +153,5 @@
     <child
       link="wheel_left_front_link" />
+    <axis xyz="0 0 1" />
   </joint>
   <link
@@ -177,5 +179,5 @@
   <joint
     name="wheel_right_back_joint"
-    type="fixed">
+    type="continuous">
     <origin
       xyz="-0.097397 -0.086125 0.04508"
@@ -185,4 +187,5 @@
     <child
       link="wheel_right_back_link" />
+    <axis xyz="0 0 1" />
   </joint>
   <link
@@ -210,5 +213,5 @@
   <joint
     name="wheel_left_back_joint"
-    type="fixed">
+    type="continuous">
     <origin
       xyz="-0.097397 0.086125 0.04508"
@@ -218,4 +221,5 @@
     <child
       link="wheel_left_back_link" />
+    <axis xyz="0 0 1" />
   </joint>
   <link

File: jetauto/jetauto_description/urdf/jetauto_flat.urdf (robot description, URDF)
Before this commit: robot jetauto, 14 links, 13 joints
Joints:
- joint wheel_left_back_joint: axis (none) -> 0 0 1; type fixed -> continuous
- joint wheel_left_front_joint: axis (none) -> 0 0 1; type fixed -> continuous
- joint wheel_right_back_joint: axis (none) -> 0 0 1; type fixed -> continuous
- joint wheel_right_front_joint: axis (none) -> 0 0 1; type fixed -> continuous
